File: STM32-NRF24L01.sch (EAGLE design)
At the start: 21 parts, among them IC1 STM32F030K6T6, IC2 MCP73811/2, IC3 SPX3819M5_3_3, J1 61301411121, J2 61301411121, P1 PUSH-SMD

Commit message: Ruteo al 50%
Connections:
- removed net PA11: IC1.PA11(CTS), J2.5
- removed net PA12: IC1.PA12(RTS), J2.6
- removed net PA8: IC1.PA8(MCO), J2.2
- net CE: now also IC1.PA12(RTS), J2.6
- net CSN: now also IC1.PA11(CTS), J2.5; no longer MOD1.CSN
- net IRQ: now also IC1.PA8(MCO), J2.2
- net NSS: now also MOD1.CSN
Changed lines of the file:
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@@
-</segment>
-</net>
-<net name="PA8" class="0">
-<segment>
-<pinref part="IC1" gate="IC$1" pin="PA8(MCO)"/>
-<wire x1="78.74" y1="78.74" x2="81.28" y2="78.74" width="0.1524" layer="91"/>
-<label x="81.28" y="78.74" size="1.27" layer="95" ratio="10" xref="yes"/>
-</segment>
-<segment>
-<pinref part="J2" gate="G$1" pin="2"/>
-<wire x1="172.72" y1="35.56" x2="172.72" y2="33.02" width="0.1524" layer="91"/>
-<label x="172.72" y="33.02" size="1.27" layer="95" ratio="10" rot="R270" xref="yes"/>
 </segment>
 </net>
@@
 </segment>
 </net>
-<net name="PA11" class="0">
-<segment>
-<pinref part="IC1" gate="IC$1" pin="PA11(CTS)"/>
-<wire x1="78.74" y1="71.12" x2="81.28" y2="71.12" width="0.1524" layer="91"/>
-<label x="81.28" y="71.12" size="1.27" layer="95" ratio="10" xref="yes"/>
-</segment>
-<segment>
-<pinref part="J2" gate="G$1" pin="5"/>
-<wire x1="165.1" y1="35.56" x2="165.1" y2="33.02" width="0.1524" layer="91"/>
-<label x="165.1" y="33.02" size="1.27" layer="95" ratio="10" rot="R270" xref="yes"/>
-</segment>
-</net>
-<net name="PA12" class="0">
-<segment>
-<pinref part="IC1" gate="IC$1" pin="PA12(RTS)"/>
-<wire x1="78.74" y1="68.58" x2="81.28" y2="68.58" width="0.1524" layer="91"/>
-<label x="81.28" y="68.58" size="1.27" layer="95" ratio="10" xref="yes"/>
-</segment>
-<segment>
-<pinref part="J2" gate="G$1" pin="6"/>
-<wire x1="162.56" y1="35.56" x2="162.56" y2="33.02" width="0.1524" layer="91"/>
-<label x="162.56" y="33.02" size="1.27" layer="95" ratio="10" rot="R270" xref="yes"/>
-</segment>
-</net>
 <net name="SWDIO" class="0">
 <segment>
@@
 <wire x1="78.74" y1="60.96" x2="81.28" y2="60.96" width="0.1524" layer="91"/>
 <label x="81.28" y="60.96" size="1.27" layer="95" ratio="10" xref="yes"/>
+</segment>
+<segment>
+<pinref part="MOD1" gate="G$1" pin="CSN"/>
+<wire x1="139.7" y1="109.22" x2="142.24" y2="109.22" width="0.1524" layer="91" style="longdash"/>
+<label x="142.24" y="109.22" size="1.27" layer="95" ratio="10" xref="yes"/>
 </segment>
 </net>
@@
 <label x="142.24" y="106.68" size="1.27" layer="95" ratio="10" xref="yes"/>
 </segment>
+<segment>
+<pinref part="IC1" gate="IC$1" pin="PA12(RTS)"/>
+<wire x1="78.74" y1="68.58" x2="81.28" y2="68.58" width="0.1524" layer="91"/>
+<label x="81.28" y="68.58" size="1.27" layer="95" ratio="10" xref="yes"/>
+</segment>
+<segment>
+<pinref part="J2" gate="G$1" pin="6"/>
+<wire x1="162.56" y1="35.56" x2="162.56" y2="33.02" width="0.1524" layer="91"/>
+<label x="162.56" y="33.02" size="1.27" layer="95" ratio="10" rot="R270" xref="yes"/>
+</segment>
 </net>
 <net name="CSN" class="0">
 <segment>
-<pinref part="MOD1" gate="G$1" pin="CSN"/>
-<wire x1="139.7" y1="109.22" x2="142.24" y2="109.22" width="0.1524" layer="91" style="longdash"/>
-<label x="142.24" y="109.22" size="1.27" layer="95" ratio="10" xref="yes"/>
+<pinref part="IC1" gate="IC$1" pin="PA11(CTS)"/>
+<wire x1="78.74" y1="71.12" x2="81.28" y2="71.12" width="0.1524" layer="91"/>
+<label x="81.28" y="71.12" size="1.27" layer="95" ratio="10" xref="yes"/>
+</segment>
+<segment>
+<pinref part="J2" gate="G$1" pin="5"/>
+<wire x1="165.1" y1="35.56" x2="165.1" y2="33.02" width="0.1524" layer="91"/>
+<label x="165.1" y="33.02" size="1.27" layer="95" ratio="10" rot="R270" xref="yes"/>
 </segment>
 </net>
@@
 <label x="142.24" y="119.38" size="1.27" layer="95" ratio="10" xref="yes"/>
 </segment>
-</net>
+<segment>
+<pinref part="IC1" gate="IC$1" pin="PA8(MCO)"/>
+<wire x1="78.74" y1="78.74" x2="81.28" y2="78.74" width="0.1524" layer="91"/>
+<label x="81.28" y="78.74" size="1.27" layer="95" ratio="10" xref="yes"/>
+</segment>
+<segment>
+<pinref part="J2" gate="G$1" pin="2"/>
+<wire x1="172.72" y1="35.56" x2="172.72" y2="33.02" width="0.1524" layer="91"/>
+<label x="172.72" y="33.02" size="1.27" layer="95" ratio="10" rot="R270" xref="yes"/>
+</segment>
+</net>
